Commit message: I don't remember what I was doing.

File: data/ur_e_description/urdf/ur5e_with_block.urdf (robot description, URDF)
Before this commit: robot ur5e, 11 links, 10 joints
Links:
- added link block, mass 0.3; collision box size=0.03 0.03 0.1; visual box size=0.03 0.03 0.1
Joints:
- added joint block-ee_fixed_joint: type fixed, parent tool0, child block, origin xyz=0 0.0 0.02 rpy=0.0 0.0 0.0
- joint wrist_3_link-tool0_fixed_joint: origin xyz=0 0 0 rpy=-1.57079632679 0 0 -> xyz=0 0.1 0 rpy=-1.57079632679 0 0

Commit message: Push all this shit. I really mast to cleaning up there

File: data/ur_e_description/urdf/ur5e_with_block.urdf (robot description, URDF)
Before this commit: robot ur5e, 12 links, 11 joints
Joints:
- joint ee_fixed_joint: origin xyz=0.0 0.1 0.0 rpy=0.0 0.0 1.57079632679 -> xyz=0.0 0.1 0.0 rpy=0.0 0.0 0.0
